Commit message: drop a similar stub geometry in the head

File: pr2_description/urdf/head_v0/head.urdf.xacro (robot description, xacro)
@@ -102,17 +102,4 @@
                  izz="0.001" />
       </inertial>
-      <visual>
-        <origin xyz="0 0 0" rpy="0 0 0" />
-        <geometry>
-          <box size="0.01 0.01 0.01" />
-        </geometry>
-        <material name="Blue" />
-      </visual>
-      <collision>
-        <origin xyz="0 0 0" rpy="0 0 0" />
-        <geometry>
-          <box size="0.01 0.01 0.01" />
-        </geometry>
-      </collision>
     </link>
     <!-- extensions -->
